File: hardware/kicad/AA-PI-Display-Board-RaspberryPi3/AA-PI-Display-Board-RaspberryPi3.sch (KiCad schematic (older format))
At the start: 100 parts, among them J1 CTP Interface, J10 MCU Interface, J11 NTC Thermistor, J12 Battery, J2 USB_B_Micro, J3 USB_B_Mini, J4 Wall adapter, J5 MCU Power, J6 LCD Interface, J7 Power Status, J8 RaspberryPi MIPI-DSI Interface, J9 VNA Board Interface, Q1 IRLML6244, Q2 IRLML2244, Q3 IRLML6244, Q4 IRLML2244, Q5 IRLML2244, Q6 IRLML2244, Q7 IRLML6244, Q8 IRLML2244, SW1 SW_SPST, SW2 SW_SPDT, U1 LTC4412, U2 AMS1117-3.3, U3 WM8731, U4 MCP73833, U5 TPS61030PWP, U6 FAN5333BSX, Y1 12.288M

Commit message: planned update (hardware)
Parts:
- added C28: 2.2u, AA-PI-Footprints:C_1206_3216Metric_Pad1.42x1.75mm_HandSolder, symbol AA-PI-Components:C_Small
- added C29: 22n, AA-PI-Footprints:C_0805_2012Metric_Pad1.15x1.40mm_HandSolder, symbol AA-PI-Components:C_Small
- added C30: 10u, AA-PI-Footprints:C_1206_3216Metric_Pad1.42x1.75mm_HandSolder, symbol AA-PI-Components:C_Small
- added C31: 100n, AA-PI-Footprints:C_0805_2012Metric_Pad1.15x1.40mm_HandSolder, symbol AA-PI-Components:C_Small
- added C32: 10u, AA-PI-Footprints:CP_EIA-3528-21_Kemet-B, symbol AA-PI-Components:CP_Small
- added Q10, Q9: IRLML6244, AA-PI-Footprints:SOT-23, symbol AA-PI-Components:N-CHANNEL-MOSFET
- added R31: 75K, AA-PI-Footprints:R_0805_2012Metric_Pad1.15x1.40mm_HandSolder, symbol AA-PI-Components:R_Small
- added R32: 0, AA-PI-Footprints:R_0805_2012Metric_Pad1.15x1.40mm_HandSolder, symbol AA-PI-Components:R_Small
- added R33, R34: 10K, AA-PI-Footprints:R_0805_2012Metric_Pad1.15x1.40mm_HandSolder, symbol AA-PI-Components:R_Small
- added R35: 500K, AA-PI-Footprints:R_0805_2012Metric_Pad1.15x1.40mm_HandSolder, symbol AA-PI-Components:R_Small
- added R36: 380K, AA-PI-Footprints:R_0805_2012Metric_Pad1.15x1.40mm_HandSolder, symbol AA-PI-Components:R_Small
- added RV1: 200K, AA-PI-Footprints:SMD-Potentiometer-Trimmer-B6W-3x3T, symbol AA-PI-Components:R_POT
- added U7: RT9193-2HPB, SOT94P279X130-5N, symbol AA-PI-Components:RT9193-2HPB
- added U8: MCP3421A0T-E_CH, AA-PI-Footprints:SOT95P280X100-6N, symbol AA-PI-Components:MCP3421A0T-E_CH
- C22, C23: value 22p -> 18p
- R14, R15: value - -> void
- U6: value FAN5333BSX -> FAN5333B
Connections:
- net +3V3: now also Q10.1 (G), Q9.1 (G); no longer L2.1, L3.1
- net +5V: now also C28.2, C31.2, C32.1, R32.1, R33.2, R34.2, U7.1 (VIN), U8.5 (VDD)
- net CHRG_STAT1: now also U4.3 (STAT1)
- net CHRG_STAT2: now also U4.4 (STAT2)
- net I2C_SCL: now also J9.3 (Pin_3), Q9.2 (S); no longer J9.4 (Pin_4)
- net I2C_SDA: now also J9.4 (Pin_4), Q10.2 (S); no longer J9.3 (Pin_3)
- net V_IN: now also U4.1 (VDD), U4.2 (VDD_1)
- net V_BATT: now reaches C27.1, J12.1 (Pin_1), Q8.3 (D)
- net V_BATT: now also U4.10 (VBAT_1), U4.9 (VBAT), R35.2
- net at C16.2, R14.1: no longer C17.2, R15.1
- net at R26.1: now also U4.8 (THERM)
- net at J11.2 (Pin_2), R25.1, R28.1: now also U4.5 (VSS)
- net at R24.2: now also U4.6 (PROG)
- net RADIO_EN: now reaches J9.6 (Pin_6)
- net RADIO_EN: now also J10.8 (Pin_8)
- net at U4.7 (~PG): now also Q7.3 (D), R21.2
- net ADC_EN: now reaches J10.7 (Pin_7)
- net ADC_EN: now also R31.1, R32.2, U7.3 (EN)
- net at U5.17 (EP), U5.3 (PGND), U5.4 (PGND_1)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: no longer C10.2, R19.1
- new net: C17.2, R15.1
- new net: C31.1, C32.2
- new net: C29.2, U7.2 (GND)
- new net: C29.1, U7.4 (BP)
- new net: R35.1, R36.2, U8.1 (VIN+)
- new net: C10.2, R19.1
- new net: R36.1, RV1.2, RV1.3
- new net I2C_SCL_H: Q9.3 (D), R34.1, U8.3 (SCL)
- new net I2C_SDA_H: Q10.3 (D), R33.1, U8.4 (SDA)
- new net V_ADC: C30.2, L2.1, L3.1, U7.5 (VOUT)
Other:
- moved on the sheet: C1, C10, C11, C12, C13, C14, C15, C16, C17, C18, C19, C2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
