File: hardware/kicad/AA-PI-Radio-Board/AA-PI-Radio-Board.sch (KiCad schematic (older format))
At the start: 74 parts, among them J1 ANT-IN, J2 MAIN BOARD, J3 INDUCT, J4 INDUCT, J5 WORK, J6 HWCAL, J7 V/I OUT, U1 Si5351A, U2 SA612A, U3 SA612A, U4 RT9193-33GB, U5 MC4558, Y1 27M

Commit message: planned update (hardware)
Parts:
- removed C16: 10u, AA-PI-Footprints:CP_EIA-3528-21_Kemet-B, symbol AA-PI-Components:CP_Small
- removed J5: WORK, AA-PI-Footprints:PinHeader_1x02_P2.54mm_Vertical, symbol AA-PI-Components:Conn_01x02
- removed J6: HWCAL, AA-PI-Footprints:PinHeader_1x02_P2.54mm_Vertical, symbol AA-PI-Components:Conn_01x02
- added C16: 4.7u, AA-PI-Footprints:C_0805_2012Metric_Pad1.15x1.40mm_HandSolder, symbol AA-PI-Components:C_Small
- added R23: 100K, AA-PI-Footprints:R_0805_2012Metric_Pad1.15x1.40mm_HandSolder, symbol AA-PI-Components:R_Small
- added R24: 0, AA-PI-Footprints:R_0805_2012Metric_Pad1.15x1.40mm_HandSolder, symbol AA-PI-Components:R_Small
- added SW1: HWCAL/WORK, AA-PI-Footprints:SW_SPDT_PCM12, symbol AA-PI-Components:SW_SPDT
Connections:
- net +5V: now also C16.2, R24.2; no longer U4.3 (EN)
- net at R4.2: now also SW1.2 (B)
- net at R9.1: now also SW1.1 (A)
- net at J4.1 (In): now also SW1.3 (C)
- net RADIO_EN: now reaches J2.6 (Pin_6)
- net RADIO_EN: now also U4.3 (EN), R23.2, R24.1
Other:
- moved on the sheet: C10, C11, C19, C23, C3, C4, C9, L1, R15, R16, R3, U4
