File: hardware/kicad/EV2400/EV2400-EVM-Interface-Board/EV2400-EVM-Interface-2.sch (KiCad schematic (older format))
At the start: 75 parts, among them J2 Conn_01x04, J3 Conn_01x04, J4 Conn_01x04, J5 Conn_01x04, Q1 BSS209PW, Q2 BSS209PW, Q3 BSS209PW, Q4 BSS209PW, Q5 BSS209PW, Q6 BSS209PW, Q7 2N7002W, Q8 2N7002W, Q9 2N7002W, U3 TPS76333DBV, U4 ST2329BQTR, U5 ST2329BQTR, U6 ST2329BQTR, U7 TPS79650DCQ, U8 TPS2113APWR

Commit message: EV2400 PCB update
Connections:
- net GND: now also C11.2, U8.5 (GND)
- net at D3.1, J3.3 (Pin_3), R14.2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: no longer D4.1
- net at J3.2 (Pin_2), R13.2, R17.2: now also D4.1
Other:
- moved on the sheet: C12
Changed lines of the file:
@@
 	10900 3070 10900 3200
 Connection ~ 10900 3200
-Wire Wire Line
-	10900 3200 11900 3200
 $Comp
 L EV2400-Components:R_Small R14
@@
 	10700 3350 10700 3300
 Connection ~ 10700 3300
-Wire Wire Line
-	10700 3300 11200 3300
-Wire Wire Line
-	11200 3350 11200 3300
-Connection ~ 11200 3300
-Wire Wire Line
-	11200 3300 11500 3300
 $Comp
 L EV2400-Components:TPS2113APWR U8
@@
 	8000 6300 8000 5980
 Wire Wire Line
-	8100 6200 8100 6380
+	8200 6200 8200 6380
 $Comp
 L EV2400-Components:C_Small C12
 U 1 1 5D9C403C
-P 8100 6480
-F 0 "C12" H 8140 6560 50  0000 L CNN
-F 1 "4.7u" H 8140 6390 50  0000 L CNN
-F 2 "EV2400-Footprints:C_0805_2012Metric" H 8100 6480 50  0001 C CNN
-F 3 "~" H 8100 6480 50  0001 C CNN
-	1    8100 6480
+P 8200 6480
+F 0 "C12" H 8240 6560 50  0000 L CNN
+F 1 "4.7u" H 8240 6390 50  0000 L CNN
+F 2 "EV2400-Footprints:C_0805_2012Metric" H 8200 6480 50  0001 C CNN
+F 3 "~" H 8200 6480 50  0001 C CNN
+	1    8200 6480
 	1    0    0    -1
 $EndComp
@@
 	6600 6630 6600 6800
 Wire Wire Line
-	6600 6800 8100 6800
-Wire Wire Line
-	8100 6800 8100 6580
-Wire Wire Line
-	8100 6200 8200 6200
-Connection ~ 8100 6200
+	6600 6800 8000 6800
+Wire Wire Line
+	8200 6800 8200 6580
+Wire Wire Line
+	8200 6200 8300 6200
+Connection ~ 8200 6200
 $Comp
 L EV2400-Components:+V_USB #PWR0139
 U 1 1 5D9DB52A
-P 8200 6200
-F 0 "#PWR0139" H 8200 6050 50  0001 C CNN
-F 1 "+V_USB" V 8200 6328 50  0000 L CNN
-F 2 "" H 8200 6200 50  0001 C CNN
-F 3 "" H 8200 6200 50  0001 C CNN
-	1    8200 6200
+P 8300 6200
+F 0 "#PWR0139" H 8300 6050 50  0001 C CNN
+F 1 "+V_USB" V 8300 6328 50  0000 L CNN
+F 2 "" H 8300 6200 50  0001 C CNN
+F 3 "" H 8300 6200 50  0001 C CNN
+	1    8300 6200
 	0    1    1    0
 $EndComp
@@
 Wire Wire Line
 	9200 6600 9200 6420
-Wire Wire Line
-	8100 6800 9000 6800
-Wire Wire Line
-	9000 6800 9000 7000
-Wire Wire Line
-	9000 7000 9100 7000
-Connection ~ 8100 6800
+Connection ~ 8200 6800
 Wire Wire Line
 	9100 6600 9100 7000
@@
 	7600 6100 8500 6100
 Wire Wire Line
-	7600 6200 8100 6200
+	7600 6200 8200 6200
 Wire Wire Line
 	7600 6300 8000 6300
@@
 Wire Wire Line
 	6100 8900 6300 8900
+Wire Wire Line
+	8000 6300 8000 6800
+Connection ~ 8000 6300
+Connection ~ 8000 6800
+Wire Wire Line
+	8000 6800 8200 6800
+Wire Wire Line
+	9000 7000 9100 7000
+Wire Wire Line
+	9000 6800 9000 7000
+Wire Wire Line
+	8200 6800 9000 6800
+Wire Wire Line
+	10700 3300 11500 3300
+Wire Wire Line
+	10900 3200 11200 3200
+Wire Wire Line
+	11200 3350 11200 3200
+Connection ~ 11200 3200
+Wire Wire Line
+	11200 3200 11900 3200
 $EndSCHEMATC
