File: hardware/kicad/EV2400/EV2400-EVM-Interface-Board/EV2400-EVM-Interface-Board.kicad_pcb (KiCad board)
At the start: 2 copper layers, 102.1 x 68.8 mm, 155 parts, among them J1 USB Connector, J2 Conn_01x04, J3 Conn_01x04, J4 Conn_01x04, J5 Conn_01x04, J6 Conn_02x12_Odd_Even, J7 Wall adapter, J8 JTAG/SBW, Q1 BSS209PW, Q2 BSS209PW, Q3 BSS209PW, Q4 BSS209PW, Q5 BSS209PW, Q6 BSS209PW, Q7 2N7002W, Q8 2N7002W, Q9 2N7002W, U1 MSP430F5529IPNR, U10 TPS73601DBV, U11 TPS73601DBV, U12 TPS73601DBV, U13 TPS73601DBV, U14 ISL90842UIV1427Z, U15 TPS73601DBV, U18 TPS73601DBV, U2 TPS2550DBV, U3 TPS76333DBV, U4 ST2329BQTR, U5 ST2329BQTR, U6 ST2329BQTR, U7 TPS79650DCQ, U8 TPS2113APWR, U9 ISL90842UIV1427Z, Y1 4MHz

Commit message: EV2400 PCB update
Parts:
- removed the REF** at (200.2, 134.4)
- moved C9 5.51 mm to (168.8, 123.6)
- moved TP2 4.58 mm to (175.2, 111.3)
- moved R19 4.37 mm to (181.7, 88.3)
- moved C23 3.22 mm to (162.7, 93.2)
- moved R30 3.21 mm to (164.3, 93.2)
- moved R21 3.17 mm to (163.3, 69.2)
- moved C34 3.05 mm to (153.3, 90.0)
- moved R10 3.02 mm to (139.6, 69.2)
- moved R8 2.98 mm to (141.3, 69.2)
- moved U13 2.97 mm to (166.8, 92.8)
- moved R5 2.96 mm to (153.3, 88.2)
- moved U14 2.92 mm to (152.6, 101.6)
- moved C35 2.90 mm to (153.2, 96.4)
- moved C30 2.87 mm to (158.5, 96.4)
- moved Q1 2.86 mm to (140.4, 65.4)
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Connections:
- C11 pad 2: Net-(C11-Pad2) -> GND
- D4 pad 1: Net-(D3-Pad1) -> Net-(D4-Pad1)
- J3 pad 2: Net-(J3-Pad2) -> Net-(D4-Pad1)
- R13 pad 2: Net-(J3-Pad2) -> Net-(D4-Pad1)
- R17 pad 2: Net-(J3-Pad2) -> Net-(D4-Pad1)
- U8 pad 5: Net-(C11-Pad2) -> GND
Routing:
- net +3V3: track 84.1 -> 280.5 mm, vias 3 -> 17
- net 5V-MUX: track 0.00 -> 147.4 mm, vias 0 -> 8
- net VPUV.1: track 0.00 -> 145.3 mm, vias 0 -> 5
- net VVOD.3: track 0.00 -> 128.9 mm, vias 0 -> 2
- net Net-(JP6-Pad2): track 0.00 -> 115.5 mm, vias 0 -> 3
- net VVOD.4: track 0.00 -> 112.1 mm, vias 0 -> 3
- net VVOD.1: track 0.00 -> 103.9 mm, vias 0 -> 3
- net SW.1: track 2.20 -> 103.9 mm, vias 1 -> 4
- net Net-(JP5-Pad2): track 0.00 -> 97.8 mm, vias 0 -> 3
- net SW.2: track 2.22 -> 99.0 mm, vias 1 -> 4
- net P6.5: track 0.00 -> 92.0 mm, vias 0 -> 1
- net SWPUE: track 3.70 -> 93.1 mm, vias 1 -> 3
- net +V_USB: track 17.0 -> 104.5 mm, vias 0 -> 2
- net P6.7: track 0.00 -> 85.0 mm, vias 0 -> 2
- net P6.6: track 0.00 -> 83.1 mm, vias 0 -> 1
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- added copper zone on B.Cu, net +3V3
- added copper zone on F.Cu, net +3V3
- added copper zone on F.Cu, net +V_PLUG
- added copper zone on F.Cu, net 5V-MUX
- added copper zone on B.Cu, net GND
- added copper zone on F.Cu, net GND
- added copper zone on F.Cu, net Net-(C11-Pad1)
