File: hardware/kicad/EV2400/EV2400-EVM-Interface-Board/EV2400-EVM-Interface-Board.kicad_pcb (KiCad board)
At the start: 2 copper layers, 102.1 x 68.8 mm, 154 parts, among them J1 USB Connector, J2 Conn_01x04, J3 Conn_01x04, J4 Conn_01x04, J5 Conn_01x04, J6 Conn_02x12_Odd_Even, J7 Wall adapter, J8 JTAG/SBW, Q1 BSS209PW, Q2 BSS209PW, Q3 BSS209PW, Q4 BSS209PW, Q5 BSS209PW, Q6 BSS209PW, Q7 2N7002W, Q8 2N7002W, Q9 2N7002W, U1 MSP430F5529IPNR, U10 TPS73601DBV, U11 TPS73601DBV, U12 TPS73601DBV, U13 TPS73601DBV, U14 ISL90842UIV1427Z, U15 TPS73601DBV, U18 TPS73601DBV, U2 TPS2550DBV, U3 TPS76333DBV, U4 ST2329BQTR, U5 ST2329BQTR, U6 ST2329BQTR, U7 TPS79650DCQ, U8 TPS2113APWR, U9 ISL90842UIV1427Z, Y1 4MHz

Commit message: Update kikad files
Parts:
- moved C3 0.40 mm to (169.8, 86.1)
Connections:
- D1 pad 3: Net-(D1-Pad3) -> unconnected-(D1-NC-Pad3)
- D2 pad 3: Net-(D2-Pad3) -> unconnected-(D2-NC-Pad3)
- D3 pad 3: Net-(D3-Pad3) -> unconnected-(D3-NC-Pad3)
- D4 pad 3: Net-(D4-Pad3) -> unconnected-(D4-NC-Pad3)
- D5 pad 3: Net-(D5-Pad3) -> unconnected-(D5-NC-Pad3)
- D6 pad 3: Net-(D6-Pad3) -> unconnected-(D6-NC-Pad3)
- U1 pad 10: Net-(U1-Pad10) -> unconnected-(U1-P5.1/A9/VREF-/VEREF--Pad10)
- U1 pad 12: Net-(U1-Pad12) -> unconnected-(U1-P5.4/XIN-Pad12)
- U1 pad 13: Net-(U1-Pad13) -> unconnected-(U1-P5.5/XOUT-Pad13)
- U1 pad 26: Net-(U1-Pad26) -> unconnected-(U1-P1.5/TA0.4-Pad26)
- U1 pad 27: Net-(U1-Pad27) -> unconnected-(U1-P1.6/TA1CLK/CBOUT-Pad27)
- U1 pad 28: Net-(U1-Pad28) -> unconnected-(U1-P1.7/TA1.0-Pad28)
- U1 pad 32: Net-(U1-Pad32) -> unconnected-(U1-P2.3/TA2.0-Pad32)
- U1 pad 33: Net-(U1-Pad33) -> unconnected-(U1-P2.4/TA2.1-Pad33)
- U1 pad 34: Net-(U1-Pad34) -> unconnected-(U1-P2.5/TA2.2-Pad34)
- U1 pad 5: Net-(U1-Pad5) -> unconnected-(U1-P7.0/CB8/A12-Pad5)
- U1 pad 55: Net-(U1-Pad55) -> unconnected-(U1-P5.6/TB0.0-Pad55)
- U1 pad 56: Net-(U1-Pad56) -> unconnected-(U1-P5.7/TB0.1-Pad56)
- U1 pad 6: Net-(U1-Pad6) -> unconnected-(U1-P7.1/CB9/A13-Pad6)
- U1 pad 7: Net-(U1-Pad7) -> unconnected-(U1-P7.2/CB10/A14-Pad7)
- U1 pad 72: Net-(U1-Pad72) -> unconnected-(U1-PJ.0/TDO-Pad72)
- U1 pad 73: Net-(U1-Pad73) -> unconnected-(U1-PJ.1/TDI/TCLK-Pad73)
- U1 pad 74: Net-(U1-Pad74) -> unconnected-(U1-PJ.2/TMS-Pad74)
- U1 pad 75: Net-(U1-Pad75) -> unconnected-(U1-PJ.3/TCK-Pad75)
- U1 pad 8: Net-(U1-Pad8) -> unconnected-(U1-P7.3/CB11/A15-Pad8)
- U1 pad 9: Net-(U1-Pad9) -> unconnected-(U1-P5.0/A8/VREF+/VEREF+-Pad9)
- U14 pad 1: Net-(U14-Pad1) -> unconnected-(U14-RH3-Pad1)
- U14 pad 2: Net-(U14-Pad2) -> unconnected-(U14-RW3-Pad2)
- U14 pad 8: Net-(U14-Pad8) -> unconnected-(U14-RW1-Pad8)
- U14 pad 9: Net-(U14-Pad9) -> unconnected-(U14-RH1-Pad9)
- U2 pad 4: Net-(U2-Pad4) -> unconnected-(U2-~{FAULT}-Pad4)
- U3 pad 4: Net-(U3-Pad4) -> unconnected-(U3-NC/FB-Pad4)
Routing:
- net Net-(J1-Pad5): track 15.5 -> 29.0 mm
- net GND: track 35.9 -> 39.0 mm, vias 99 -> 115
- net Net-(JP5-Pin_2): track 97.8 -> 99.9 mm
- net VVOD.2: track 82.8 -> 80.9 mm
- net +V_USB: track 104.5 -> 106.1 mm
- net SW.2: track 99.0 -> 99.8 mm
- net +3V3: track 280.5 -> 279.8 mm
Other:
- net class Default removed
- net class Power removed
