File: hardware/kicad/EV2400/EV2400-EVM-Interface-Board/EV2400-EVM-Interface-Board.kicad_sch (KiCad schematic)
At the start: 39 parts, among them J1 USB Connector, J6 Conn_02x12_Odd_Even, J7 Wall adapter, J8 JTAG/SBW, U1 MSP430F5529IPNR, U2 TPS2550DBV, Y1 4MHz

Commit message: Update EV2400 kicad files
Parts:
- C13, C36, C37, C38, C39, C40, C41, C42, C43: symbol Dreamstalker-Components:C_Small -> EV2400-Components:C_Small
- C9: symbol EV2400-EVM-Interface-Board-rescue:CP_Small-EV2400-Components -> EV2400-Components:CP_Small
- D7, D8, D9: symbol EV2400-EVM-Interface-Board-rescue:LED_ALT-EV2400-Components -> EV2400-Components:LED_ALT
- E1, E2, E3, E4: symbol EV2400-EVM-Interface-Board-rescue:TestPoint_Alt-EV2400-Components -> EV2400-Components:TestPoint_Alt
- J1: symbol EV2400-EVM-Interface-Board-rescue:USB_B-EV2400-Components -> EV2400-Components:USB_B
- J6: symbol EV2400-EVM-Interface-Board-rescue:Conn_02x12_Odd_Even-EV2400-Components -> EV2400-Components:Conn_02x12_Odd_Even
- J7: symbol EV2400-EVM-Interface-Board-rescue:Barrel_Jack_Switch-EV2400-Components -> EV2400-Components:Barrel_Jack_Switch
- J8: symbol EV2400-EVM-Interface-Board-rescue:Conn_01x04-EV2400-Components -> EV2400-Components:Conn_01x04
- JP7: symbol EV2400-EVM-Interface-Board-rescue:Conn_02x01-EV2400-Components -> EV2400-Components:Conn_02x01
- R1, R2, R27, R3, R39, R4, R40, R41, R42: symbol Dreamstalker-Components:R_Small -> EV2400-Components:R_Small
- SW1: symbol Dreamstalker-Components:SW_Push -> EV2400-Components:SW_Push
- TP1, TP2, TP3, TP4: symbol EV2400-EVM-Interface-Board-rescue:TestPoint-EV2400-Components -> EV2400-Components:TestPoint
- U1: symbol EV2400-EVM-Interface-Board-rescue:MSP430F5529IPNR-EV2400-Components -> EV2400-Components:MSP430F5529IPNR; Description_1 (none) -> 16-Bit Ultra-Low-Power Microcontroller, 128KB Flash, 8KB RA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
- U2: symbol EV2400-EVM-Interface-Board-rescue:TPS2550DBV-EV2400-Components -> EV2400-Components:TPS2550DBV; Description_1 (none) -> Texas Instruments TPS2550DBVT, USB Power Switch High Side, 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
- Y1: symbol EV2400-EVM-Interface-Board-rescue:Crystal-EV2400-Components -> EV2400-Components:Crystal
