File: hardware/kicad/AA-PI/AA-PI-V4_0-Radio-Board/AA-PI-V4-Radio-Board.kicad_pcb (KiCad board)
At the start: 2 copper layers, 56 x 65 mm, 80 parts, among them J1 ANT-IN, J2 Main Board, J3 INDUCT, J4 INDUCT, U1 Si5351A, U2 SA612A, U3 SA612A, U5 MC4558, Y1 27M

Commit message: Updated to v4.3
Changed lines of the file:
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@@
 		(tags "capacitor handsolder")
 		(property "Reference" "C1"
-			(at 2.55 0 0)
+			(at 2.58 -0.04 0)
 			(layer "F.SilkS")
 			(effects
@@
 		(tags "capacitor handsolder")
 		(property "Reference" "C2"
-			(at 2.6 0 0)
+			(at -2.67 -0.03 0)
 			(layer "F.SilkS")
 			(effects
@@
 		(tags "capacitor handsolder")
 		(property "Reference" "C6"
-			(at 1.23 -2.02 0)
+			(at 0.3 -2.06 0)
 			(layer "F.SilkS")
 			(effects
@@
 		(tags "resistor handsolder")
 		(property "Reference" "R6"
-			(at 2.81 0.03 0)
+			(at 2.96 0.02 0)
 			(layer "F.SilkS")
 			(effects
@@
 		(tags "Integrated Circuit")
 		(property "Reference" "U1"
-			(at 3.97 1.46 0)
+			(at 2.75 -2.98 0)
 			(layer "F.SilkS")
 			(effects
@@
 		(tags "SMD SMT crystal")
 		(property "Reference" "Y1"
-			(at 1.13 3.02 180)
+			(at -0.37 -2.86 180)
 			(layer "F.SilkS")
 			(effects
@@
 		(tags "test point THT pad")
 		(property "Reference" "TP4"
-			(at -0.21 -1.48 0)
+			(at -0.17 -1.52 0)
 			(layer "F.SilkS")
 			(effects
