File: hardware/kicad/AA-PI/AA-PI-V4_0-Radio-Board/AA-PI-V4-Radio-Board.kicad_sch (KiCad schematic)
At the start: 73 parts, among them J1 ANT-IN, J2 Main Board, J3 INDUCT, J4 INDUCT, U1 Si5351A, U2 SA612A, U3 SA612A, U5 MC4558, Y1 27M

Commit message: Planned updates: radio board design files
Parts:
- C32, C33: value 10u -> 100n
- R17, R18, R19, R21: value 12K -> 7.5K
