File: hardware/kicad/AA-PI/AA-PI-V4_0-Display-Board-BananapiM2M/AA-PI-V4-Display-Board-BananapiM2M-LCD-CTP.kicad_sch (KiCad schematic)
At the start: 22 parts, among them J7 BananaPi M2M Interface, J8 FS050HD020-C020C, J9 FS050HD020-C020C, U5 TCA9803, U6 FAN5331, U7 RT8059

Commit message: Updated to v4.3
Other:
- moved on the sheet: C18, C20, C21, L2, L3, R21, R24, R25, U7
