File: hardware/kicad/AA-PI/AA-PI-V4_0-Display-Board-BananapiM2M/AA-PI-V4-Display-Board-BananapiM2M-RTC.kicad_sch (KiCad schematic)
At the start: 7 parts, among them Q8 IRLML6402, U15 PCF8563TS/5,118, Y2 32.768KHz

Commit message: Planned updates: display board design files
Other:
- moved on the sheet: C38
