File: hardware/kicad/AA-PI/AA-PI-V4_0-Display-Board-BananapiM2M/AA-PI-V4-Display-Board-BananapiM2M-VNA-Codec.kicad_sch (KiCad schematic)
At the start: 39 parts, among them J10 VNA Board Interface, U10 TCA9803, U11 SI5351A-B-GM1, U12 TPS2051BDBVR, U8 RT9193-2HPB, U9 PCM1803A, Y1 24.576MHz

Commit message: Updated to v4.3
Parts:
- removed U11: SI5351A-B-GM1, AA-PI-Footprints:QFN50P300X300X90-17N-D, symbol AA-PI-Components:SI5351A-B-GM1
- added U11: Si5351A-B-GM, AA-PI-Footprints:QFN50P400X400X90-21N-D, symbol AA-PI-Components:Si5351A-B-GM
Connections:
- net +VDD_RADIO: now also U11.10 (VDDOB), U11.11 (VDDOA), U11.14 (VDDOD), U11.18 (VDDOC), U11.20 (VDD)
- net ADC_CLK1: now also U11.13 (CLK0)
- net GND: now also U11.21 (GND), U11.6 (SSEN), U11.7 (OEB)
- net VNA_I2C_SCL: now also U11.4 (SCL)
- net VNA_I2C_SDA: now also U11.5 (SDA)
- net at C53.1, Y1.1: now also U11.2 (XB)
- net at C54.1, Y1.2: now also U11.1 (XA)
- net at R53.2, R54.2: now also U11.3 (A0)
Other:
- moved on the sheet: C53, C54, C55, R53, R54

Commit message: Planned updates: display board design files
Parts:
- removed C52: 100n, AA-PI-Footprints:C_0603_1608Metric, symbol AA-PI-Components:C_Small
- removed U11: Si5351A-B-GM, AA-PI-Footprints:QFN50P400X400X90-21N-D, symbol AA-PI-Components:Si5351A-B-GM
- removed U8: RT9193-2HPB, AA-PI-Footprints:SOT94P279X130-5N, symbol AA-PI-Components:RT9193-2HPB
- added R55, R56, R57, R58: 0, AA-PI-Footprints:R_0603_1608Metric, symbol AA-PI-Components:R_Small
- added U11: ICS512M, SOIC127P600X175-8N, symbol AA-PI-Components:ICS512M
- added U8: RT9193-33GB, SOT94P279X130-5N, symbol AA-PI-Components:RT9193-33GB
- C53, C54: value 100n -> 22p
- R53, R54: value 0 -> 33
Connections:
- net +5V: now also U8.1 (VIN)
- net +VDD_RADIO: now also R55.2, R57.2, U11.2 (VDD), U8.5 (VOUT); no longer R54.1
- net ADC_CLK1: now also R53.2, R54.2
- net GND: now also R56.2, R58.2, U11.3 (GND), U8.2 (GND); no longer R53.1
- net RADIO_EN: now also U8.3 (EN)
- net at C53.1, Y1.1: now also U11.1 (X1/ICLK)
- net at C54.1, Y1.2: now also U11.8 (X2)
- net at C31.1: now also U8.4 (BP)
- new net: R55.1, R56.1, U11.7 (S1)
- new net: R57.1, R58.1, U11.6 (S0)
- new net: R54.1, U11.4 (REF)
- new net: R53.1, U11.5 (CLK)
Other:
- note added: "VNA Codec Dedicated Clock"
- note removed: "I2C Addr Selection: A0 low => 0x60 A0 high => 0x61"
- note removed: "VNA Codec Clock"
- moved on the sheet: C53, C54, C55, R51, R52, R53, R54, Y1
