File: hardware/kicad/AA-PI/AA-PI-V4_0-Display-Board-BananapiM2M/AA-PI-V4-Display-Board-BananapiM2M.kicad_pcb (KiCad board)
At the start: 2 copper layers, 140 x 85 mm, 184 parts, among them J1 Wall adapter, J10 VNA Board Interface, J11 Battery Pack, J2 USB_C_Power, J3 USB_B_Mini, J4 MCU GPIO, J5 MCU Power, J6 MCU UART, J7 BananaPi M2M Interface, J8 FS050HD020-C020C, J9 FS050HD020-C020C, K1 CPC1117N, Q1 Si2333CDS, Q2 Si2333CDS, Q3 IRLML2402, Q4 Si2333CDS, Q5 IRLML6402, Q6 IRLML2402, Q7 Si2333CDS, Q8 IRLML6402, SW1 ON/OFF, SW2 SW_Push, U1 LTC2951-2, U10 TCA9803, U11 SI5351A-B-GM1, U12 TPS2051BDBVR, U13 SN74HC164PW, U14 BQ34Z100-G1, U15 PCF8563TS/5,118, U2 LTC4412, U3 MAX1709ESE, U4 MCP73833, U5 TCA9803, U6 FAN5331, U7 RT8059, U8 RT9193-2HPB, U9 PCM1803A, Y1 24.576MHz, Y2 32.768KHz

Commit message: Updated to v4.3
Parts:
- removed C36: 2.2u, AA-PI-Footprints:C_0805_2012Metric_Pad1.15x1.40mm_HandSolder
- removed C36: 1u, AA-PI-Footprints:C_0603_1608Metric
- added D20: 1N4148, AA-PI-Footprints:D_SOD-323_HandSoldering, F.Cu at (108.7, 117.3)
- added D21: Wall adapter, AA-PI-Footprints:LED_0805_2012Metric_Pad1.15x1.40mm_HandSolder, F.Cu at (92.9, 119.3)
- added R45: 33K, AA-PI-Footprints:R_0603_1608Metric, F.Cu at (133.6, 107.3)
- C15: value 100n -> 22n
- C8: value 330n -> 220n
- D1, D2, D5, D7: value SS54 -> SS34; footprint AA-PI-Footprints:D_SMB -> AA-PI-Footprints:D_SMA
- D6: value Wall adapter -> SS34; footprint AA-PI-Footprints:LED_0805_2012Metric_Pad1.15x1.40mm_HandSolder -> AA-PI-Footprints:D_SMA
- Q2: value Si2333CDS -> IRLML2402
- R16: value 1K -> 2K
- R29: value 10K -> 100K
- R32: value 100 -> 47K
- R5: value 75K -> 100K
- U11: value SI5351A-B-GM1 -> Si5351A-B-GM; footprint AA-PI-Footprints:QFN50P300X300X90-17N-D -> AA-PI-Footprints:QFN50P400X400X90-21N-D
- moved Q2 46.5 mm to (132.5, 110.8)
- moved R35 11.4 mm to (100.3, 97.8)
- moved D6 8.99 mm to (87.9, 126.7), turned to -90 degrees
- moved R5 6.18 mm to (104.4, 121.1)
- moved C15 5.81 mm to (106.0, 121.1), turned to 90 degrees
- moved R32 4.63 mm to (108.2, 115.4)
- moved F1 2.12 mm to (88.2, 133.4)
- moved D3 1.26 mm to (83.8, 128.0)
- moved C52 1.17 mm to (71.8, 111.3)
- moved C55 1.08 mm to (63.0, 113.2)
- moved R9 1.07 mm to (112.5, 122.3)
- moved U11 0.59 mm to (67.4, 111.3)
- moved R46 0.46 mm to (132.5, 116.7)
- moved R16 0.37 mm to (88.7, 99.2)
- moved R15 0.27 mm to (100.3, 99.5)
Connections:
- C15 pad 1: Net-(C15-Pad1) -> +V_BAT
- C15 pad 2: +V_LOAD -> Net-(D20-K)
- D6 pad 1: Net-(D6-K) -> +V_IN
- D6 pad 2: Net-(D6-A) -> /V_SUPPLY
- J4 pad 26: ~{CHRG_FAST} -> CHRG_FAST
- K1 pad 3: ~{CHRG_FAST} -> GND
- Q2 pad 1: Net-(Q2-G) -> CHRG_FAST
- Q2 pad 2: +V_IN -> GND
- Q2 pad 3: /V_SUPPLY -> Net-(Q2-D)
- Q4 pad 1: Net-(Q4-G) -> Net-(D20-K)
- Q5 pad 1: Net-(Q2-G) -> Net-(Q5-G)
- Q5 pad 3: Net-(D6-A) -> Net-(D21-A)
- R32 pad 1: Net-(Q4-G) -> Net-(D20-A)
- R32 pad 2: Net-(C15-Pad1) -> Net-(D20-K)
- R35 pad 1: GND -> Net-(U4-PROG)
- R35 pad 2: ~{CHRG_FAST} -> Net-(Q2-D)
- R4 pad 1: Net-(Q2-G) -> Net-(Q5-G)
- R5 pad 1: Net-(Q4-G) -> +V_BAT
- R5 pad 2: Net-(U1-EN/~{EN}) -> Net-(D20-A)
- R7 pad 2: Net-(D6-K) -> Net-(D21-K)
- U1 pad 6: Net-(U1-EN/~{EN}) -> Net-(D20-A)
- U11 pad 10: ADC_CLK1 -> +VDD_RADIO
- U11 pad 13: unconnected-(U11-CLK2-Pad13) -> ADC_CLK1
- U11 pad 15: GND -> unconnected-(U11-CLK7-Pad15)
- U11 pad 16: +VDD_RADIO -> unconnected-(U11-CLK6-Pad16)
- U11 pad 17: GND -> unconnected-(U11-CLK5-Pad17)
- U11 pad 7: unconnected-(U11-CLK1-Pad7) -> GND
- U11 pad 8: +VDD_RADIO -> unconnected-(U11-CLK3-Pad8)
- U11 pad 9: +VDD_RADIO -> unconnected-(U11-CLK2-Pad9)
- U2 pad 4: Net-(Q2-G) -> Net-(Q5-G)
- U3 pad 16: Net-(U1-EN/~{EN}) -> Net-(D20-A)
Routing:
- net ~{CHRG_FAST}: track 56.9 -> 0.00 mm, vias 4 -> 0
- net Net-(D20-A): track 0.00 -> 56.7 mm, vias 0 -> 3
- net Net-(U1-EN/~{EN}): track 49.9 -> 0.00 mm, vias 3 -> 0
- net Net-(Q2-D): track 0.00 -> 40.5 mm, vias 0 -> 2
- net Net-(Q2-G): track 15.1 -> 0.00 mm, vias 3 -> 0
- net Net-(Q5-G): track 0.00 -> 14.6 mm, vias 0 -> 2
- net Net-(U4-PROG): track 9.82 -> 23.2 mm
- net Net-(D20-K): track 0.00 -> 9.11 mm
- net VNA_I2C_SCL: track 65.3 -> 72.5 mm
- net Net-(Q4-G): track 7.10 -> 0.00 mm
- net GND: track 17.3 -> 11.8 mm, vias 151 -> 152
- net CHRG_FAST: track 0.00 -> 5.19 mm
- net Net-(D21-A): track 0.00 -> 3.77 mm
- net Net-(D6-A): track 3.75 -> 0.00 mm
- net Net-(D6-K): track 3.19 -> 0.00 mm
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
Commit message: Planned updates: display board design files
Parts:
- removed C52: 100n, AA-PI-Footprints:C_0603_1608Metric
- added R55: 0, AA-PI-Footprints:R_0603_1608Metric, F.Cu at (62.8, 106.6)
- added R56: 0, AA-PI-Footprints:R_0603_1608Metric, F.Cu at (73.8, 108.4)
- added R57: 0, AA-PI-Footprints:R_0603_1608Metric, F.Cu at (62.8, 113.7)
- added R58: 0, AA-PI-Footprints:R_0603_1608Metric, F.Cu at (73.8, 111.9)
- U11: value Si5351A-B-GM -> ICS512M; footprint AA-PI-Footprints:QFN50P400X400X90-21N-D -> AA-PI-Footprints:SOIC127P600X175-8N
- U8: value RT9193-2HPB -> RT9193-33GB
- moved R53 18.2 mm to (72.4, 114.5), turned to -45 degrees
- moved R54 12.6 mm to (67.0, 114.5), turned to -45 degrees
- moved C55 2.98 mm to (63.8, 110.3), turned to 90 degrees
- moved U11 1.67 mm to (68.6, 110.2), turned to 0 degrees
- moved Y1 1.19 mm to (68.7, 105.1)
- moved C54 1.09 mm to (70.8, 102.1), turned to 0 degrees
- moved C53 0.92 mm to (66.4, 102.2), turned to 180 degrees
Connections:
- C53 pad 1: Net-(U11-XB) -> Net-(U11-X1/ICLK)
- C54 pad 1: Net-(U11-XA) -> Net-(U11-X2)
- R53 pad 1: GND -> Net-(U11-CLK)
- R53 pad 2: Net-(U11-A0) -> ADC_CLK1
- R54 pad 1: +VDD_RADIO -> Net-(U11-REF)
- R54 pad 2: Net-(U11-A0) -> ADC_CLK1
- U11 pad 1: Net-(U11-XA) -> Net-(U11-X1/ICLK)
- U11 pad 2: Net-(U11-XB) -> +VDD_RADIO
- U11 pad 3: Net-(U11-A0) -> GND
- U11 pad 4: VNA_I2C_SCL -> Net-(U11-REF)
- U11 pad 5: VNA_I2C_SDA -> Net-(U11-CLK)
- U11 pad 6: GND -> Net-(U11-S0)
- U11 pad 7: GND -> Net-(U11-S1)
- U11 pad 8: unconnected-(U11-CLK3-Pad8) -> Net-(U11-X2)
- Y1 pad 1: Net-(U11-XB) -> Net-(U11-X1/ICLK)
- Y1 pad 2: Net-(U11-XA) -> Net-(U11-X2)
Routing:
- net VNA_I2C_SCL: track 72.5 -> 6.08 mm
- net VNA_I2C_SDA: track 72.8 -> 6.78 mm
- net +VDD_RADIO: track 114.5 -> 82.6 mm, vias 8 -> 5
- net Net-(U11-A0): track 12.9 -> 0.00 mm
- net Net-(U11-S1): track 0.00 -> 12.0 mm, vias 0 -> 2
- net Net-(U11-S0): track 0.00 -> 11.9 mm, vias 0 -> 2
- net Net-(U11-XB): track 8.21 -> 0.00 mm
- net Net-(U11-XA): track 7.99 -> 0.00 mm
- net Net-(U11-X1/ICLK): track 0.00 -> 6.79 mm
- net Net-(U11-X2): track 0.00 -> 6.71 mm
- net Net-(U11-CLK): track 0.00 -> 2.06 mm
- net Net-(U11-REF): track 0.00 -> 2.05 mm
- net GND: vias 152 -> 149
