File: hardware/kicad/AA-PI/AA-PI-V4_0-Display-Board-BananapiM2M/AA-PI-V4-Display-Board-BananapiM2M.kicad_pcb (KiCad board)
At the start: 2 copper layers, 140 x 85 mm, 188 parts, among them J1 Wall adapter, J10 VNA Board Interface, J11 Battery Pack, J2 USB_C_Power, J3 USB_B_Mini, J4 MCU GPIO, J5 MCU Power, J6 MCU UART, J7 BananaPi M2M Interface, J8 FS050HD020-C020C, J9 FS050HD020-C020C, K1 CPC1117N, Q1 Si2333CDS, Q2 IRLML2402, Q3 IRLML2402, Q4 Si2333CDS, Q5 IRLML6402, Q6 IRLML2402, Q7 Si2333CDS, Q8 IRLML6402, SW1 ON/OFF, SW2 SW_Push, U1 LTC2951-2, U10 TCA9803, U11 ICS512M, U12 TPS2051BDBVR, U13 SN74HC164PW, U14 BQ34Z100-G1, U15 PCF8563TS/5,118, U2 LTC4412, U3 MAX1709ESE, U4 MCP73833, U5 TCA9803, U6 FAN5331, U7 RT8059, U8 RT9193-33GB, U9 PCM1803A, Y1 24.576MHz, Y2 32.768KHz

Commit message: display board design files: planned updates
Routing:
- net +VDD_RADIO: track 82.6 -> 81.3 mm
Changed lines of the file:
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@@
 		(tags "resistor")
 		(property "Reference" "R56"
-			(at -0.1475 1.5 90)
+			(at 0.0225 2.16 0)
 			(layer "F.SilkS")
 			(effects
@@
 		(tags "resistor")
 		(property "Reference" "R57"
-			(at 3.1025 -0.1 0)
+			(at 1.3725 -1.52 0)
 			(layer "F.SilkS")
 			(effects
@@
 		(tags "resistor")
 		(property "Reference" "R58"
-			(at -0.1375 -1.51 90)
+			(at 0.2125 -2.2 0)
 			(layer "F.SilkS")
 			(effects
@@
 	)
 	(segment
-		(start 57.21 105.27)
-		(end 57.21 94.17)
-		(width 0.508)
-		(layer "F.Cu")
-		(net "+VDD_RADIO")
-	)
-	(segment
 		(start 72.14 77.74)
 		(end 72.69 78.29)
@@
 	)
 	(segment
-		(start 62.045 107.955)
-		(end 62.02 107.98)
-		(width 0.508)
-		(layer "F.Cu")
-		(net "+VDD_RADIO")
-	)
-	(segment
 		(start 65.936 109.56)
 		(end 63.635 109.56)
@@
 	)
 	(segment
-		(start 77.01 78.29)
-		(end 77.735 77.565)
+		(start 62.045 106.61)
+		(end 59.79 106.61)
 		(width 0.508)
 		(layer "F.Cu")
@@
 	)
 	(segment
-		(start 78.78 76.73)
-		(end 78.78 77.42)
+		(start 77.01 78.29)
+		(end 77.735 77.565)
 		(width 0.508)
 		(layer "F.Cu")
@@
 	)
 	(segment
-		(start 59.92 107.98)
-		(end 57.21 105.27)
+		(start 78.78 76.73)
+		(end 78.78 77.42)
 		(width 0.508)
 		(layer "F.Cu")
@@
 	)
 	(segment
-		(start 62.035 111.13)
-		(end 62.035 113.71)
+		(start 59.79 106.61)
+		(end 57.21 104.03)
 		(width 0.508)
 		(layer "F.Cu")
@@
 	)
 	(segment
-		(start 66.925 87.59)
-		(end 67.31 87.59)
+		(start 62.035 111.13)
+		(end 62.035 113.71)
 		(width 0.508)
 		(layer "F.Cu")
@@
 	)
 	(segment
-		(start 62.02 107.98)
-		(end 59.92 107.98)
+		(start 66.925 87.59)
+		(end 67.31 87.59)
 		(width 0.508)
 		(layer "F.Cu")
@@
 	)
 	(segment
+		(start 57.21 104.03)
+		(end 57.21 94.17)
+		(width 0.508)
+		(layer "F.Cu")
+		(net "+VDD_RADIO")
+	)
+	(segment
 		(start 63.535 90.69)
 		(end 63.55 90.675)
@@
 		(layer "F.Cu")
 		(hatch none 0.1)
-		(priority 30008)
+		(priority 30009)
 		(attr
 			(teardrop
@@
 	)
 	(zone
+		(net "DSI_D3_N")
+		(layer "F.Cu")
+		(hatch none 0.1)
+		(priority 30007)
+		(attr
+			(teardrop
+				(type padvia)
+			)
+		)
+		(connect_pads yes
+			(clearance 0)
+		)
+		(min_thickness 0.0254)
+		(fill yes
+			(island_removal_mode 1)
+		)
+		(polygon
+			(pts
+				(xy 155.8916 70.532985) (xy 155.6884 70.532985) (xy 155.6884 70.84) (xy 155.718158 70.911842) (xy 155.705216 71.028558)
+				(xy 156.022628 71.072628) (xy 155.978558 70.755216) (xy 155.861842 70.768158)
+			)
+		)
+	)
+	(zone
 		(net "DSI_D0_N")
 		(layer "F.Cu")
@@
 		(layer "F.Cu")
 		(hatch none 0.1)
-		(priority 30009)
+		(priority 30010)
 		(attr
 			(teardrop
@@
 		(layer "F.Cu")
 		(hatch none 0.1)
-		(priority 30007)
+		(priority 30008)
 		(attr
 			(teardrop
@@
 		(layer "F.Cu")
 		(hatch none 0.1)
-		(priority 30010)
+		(priority 30011)
 		(attr
 			(teardrop
@@
 		(layer "B.Cu")
 		(hatch none 0.1)
-		(priority 30005)
+		(priority 30008)
 		(attr
 			(teardrop
@@
 		(layer "B.Cu")
 		(hatch none 0.1)
-		(priority 30007)
+		(priority 30010)
 		(attr
 			(teardrop
@@
 		(layer "B.Cu")
 		(hatch none 0.1)
-		(priority 30003)
+		(priority 30004)
 		(attr
 			(teardrop
@@
 		(layer "B.Cu")
 		(hatch none 0.1)
-		(priority 30006)
+		(priority 30009)
 		(attr
 			(teardrop
@@
 	)
 	(zone
+		(net "DSI_D3_N")
+		(layer "B.Cu")
+		(hatch none 0.1)
+		(priority 30003)
+		(attr
+			(teardrop
+				(type padvia)
+			)
+		)
+		(connect_pads yes
+			(clearance 0)
+		)
+		(min_thickness 0.0254)
+		(fill yes
+			(island_removal_mode 1)
+		)
+		(polygon
+			(pts
+				(xy 167.558941 95.359) (xy 167.558941 95.1558) (xy 167.24535 95.1558) (xy 167.173508 95.185558)
+				(xy 167.061442 95.167966) (xy 167.017372 95.485378) (xy 167.334784 95.441308) (xy 167.317192 95.329242)
+			)
+		)
+	)
+	(zone
 		(net "LED-K")
 		(layer "B.Cu")
@@
 	)
 	(zone
+		(net "DSI_CLK_N")
+		(layer "B.Cu")
+		(hatch none 0.1)
+		(priority 30006)
+		(attr
+			(teardrop
+				(type padvia)
+			)
+		)
+		(connect_pads yes
+			(clearance 0)
+		)
+		(min_thickness 0.0254)
+		(fill yes
+			(island_removal_mode 1)
+		)
+		(polygon
+			(pts
+				(xy 167.648772 98.36845) (xy 167.648772 98.16525) (xy 167.353919 98.16525) (xy 167.349626 98.165341)
+				(xy 167.086585 98.165534) (xy 167.012056 98.281307) (xy 167.399562 98.377541) (xy 167.358212 98.368359)
+			)
+		)
+	)
+	(zone
 		(net "+5V")
 		(layer "B.Cu")
@@
 		(layer "B.Cu")
 		(hatch none 0.1)
-		(priority 30008)
+		(priority 30011)
 		(attr
 			(teardrop
@@
 		(layer "B.Cu")
 		(hatch none 0.1)
-		(priority 30004)
+		(priority 30005)
 		(attr
 			(teardrop
@@
 			)
 		)
+	)
+	(zone
+		(net "DSI_D0_P")
+		(layer "B.Cu")
+		(hatch none 0.1)
+		(priority 30007)
+		(attr
+			(teardrop
+				(type padvia)
+			)
+		)
+		(connect_pads yes
+			(clearance 0)
+		)
+		(min_thickness 0.0254)
+		(fill yes
+			(island_removal_mode 1)
+		)
+		(polygon
+			(pts
+				(xy 167.608772 100.97475) (xy 167.608772 100.77155) (xy 167.318212 100.771641) (xy 167.359562 100.762459)
+				(xy 166.972056 100.858693) (xy 167.046585 100.974466) (xy 167.309626 100.974659) (xy 167.313919 100.97475)
+			)
+		)
