File: hardware/kicad/AA-PI/AA-PI-V4_0-Display-Board-BananapiM2M/AA-PI-V4-Display-Board-BananapiM2M.kicad_sch (KiCad schematic)
At the start: 73 parts, among them J1 Wall adapter, J2 USB_C_Power, J3 USB_B_Mini, J4 MCU GPIO, J5 MCU Power, J6 MCU UART, K1 CPC1117N, Q1 Si2333CDS, Q2 Si2333CDS, Q3 IRLML2402, Q4 Si2333CDS, Q5 IRLML6402, Q6 IRLML2402, Q7 Si2333CDS, SW1 ON/OFF, U1 LTC2951-2, U2 LTC4412, U3 MAX1709ESE, U4 MCP73833

Commit message: Updated to v4.3
Parts:
- removed C36: 1u, AA-PI-Footprints:C_0603_1608Metric, symbol AA-PI-Components:C_Small
- removed Q2: Si2333CDS, AA-PI-Footprints:SOT-23, symbol AA-PI-Components:P-CHANNEL-MOSFET
- added D20: 1N4148, AA-PI-Footprints:D_SOD-323_HandSoldering, symbol AA-PI-Components:D_Small
- added D6: SS34, AA-PI-Footprints:D_SMA, symbol AA-PI-Components:D_Schottky_Small
- added Q2: IRLML2402, AA-PI-Footprints:SOT-23, symbol AA-PI-Components:N-CHANNEL-MOSFET
- added R45: 33K, AA-PI-Footprints:R_0603_1608Metric, symbol AA-PI-Components:R_Small
- C15: value 100n -> 22n
- C8: value 330n -> 220n
- D1, D2, D5, D7: value SS54 -> SS34; footprint AA-PI-Footprints:D_SMB -> AA-PI-Footprints:D_SMA
- R16: value 1K -> 2K
- R29: value 10K -> 100K
- R32: value 100 -> 47K
- R5: value 75K -> 100K
- renumbered D6 to D21
Connections:
- net +V_BAT: now also C15.1, R5.1
- net +V_IN: now also D6.1 (K)
- net +V_LOAD: no longer C15.2
- net GND: now also K1.3 (LOAD1), Q2.2 (S), R45.1; no longer R35.1
- net V_SUPPLY: now also D6.2 (A)
- net at R16.2, U4.6 (PROG): now also R35.1
- net at R5.2, U1.6 (EN/~{EN}), U3.16 (~{ONB}): now also R32.1, D20.2 (A)
- net at R32.2: now also C15.2, Q4.1 (G), D20.1 (K); no longer C15.1
- removed net ~{CHRG_FAST}: J4.26 (Pin_26), K1.3 (LOAD1), R35.2
- new net: Q2.3 (D), R35.2
- new net CHRG_FAST: J4.26 (Pin_26), Q2.1 (G), R45.2
Other:
- note added: "1) The charge temperature window can be set by placing fixed value resistors in series-parallel with a thermistor. Refer to the chapter 6.1.1.6 Temperature Monitoring to find values of R17 and R18. 2) If NTC thermistor is installed then R18 is removed and R17=0 3) Charge current is controlled by R16 (2K => 500mA)"
- note added: "STAT pin goes low when the wall adapter is connected."
- note removed: "1) The charge temperature window can be set by placing fixed value resistors in series-parallel with a thermistor. Refer to the chapter 6.1.1.6 Temperature Monitoring to find values of R17 and R18. 2) If NTC thermistor is installed then R18 must be removed and R17=0 3) Charge current is controlled by R16 (2K => 500mA)"
- note removed: "The STAT pin goes low when the wall adapter is connected."
- moved on the sheet: C13, C14, C6, C8, C9, D21, D4, K1, Q3, Q4, Q5, Q6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

Commit message: Planned updates: display board design files
Other:
- note added: "Remove jumpers when the battery pack is connected to EV2400"
- note removed: "Remove jumpers to flash the battery pack"
- moved on the sheet: C13, C4, C5, C7, C8, D3, D5, D7, F1, JP1, JP2, K1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
